Commit message: xacro files rearrenged

File: description/gazebo_control.xacro (robot description, xacro)
@@ -2,38 +2,20 @@
 <robot xmlns:xacro="http://www.ros.org/wiki/xacro">
     <gazebo>
-        <plugin name="gazebo_ros_ackermann_drive" filename="libgazebo_ros_ackermann_drive.so">
-            <ros>
-                <namespace>demo</namespace>
-                <remapping>cmd_vel:=cmd_demo</remapping>
-                <remapping>odom:=odom_demo</remapping>
-                <remapping>distance:=distance_demo</remapping>
-            </ros>
-            <update_rate>100.0</update_rate>
-            <!-- wheels -->
-            <front_left_joint>front_left_wheel_joint</front_left_joint>
-            <front_right_joint>front_right_wheel_joint</front_right_joint>
-            <rear_left_joint>rear_left_wheel_joint</rear_left_joint>
-            <rear_right_joint>rear_right_wheel_joint</rear_right_joint>
-            <!-- Max absolute steer angle for tyre in radians-->
-            <!-- Any cmd_vel angular z greater than this would be capped -->
-            <max_steer>0.6458</max_steer>
-            <!-- Max absolute steering angle of steering wheel -->
-            <max_steering_angle>7.85</max_steering_angle>
-            <!-- Max absolute linear speed in m/s -->
-            <max_speed>20</max_speed>
-            <!-- PID tuning -->
-            <left_steering_pid_gain>1500 0 1</left_steering_pid_gain>
-            <left_steering_i_range>0 0</left_steering_i_range>
-            <right_steering_pid_gain>1500 0 1</right_steering_pid_gain>
-            <right_steering_i_range>0 0</right_steering_i_range>
-            <linear_velocity_pid_gain>1000 0 1</linear_velocity_pid_gain>
-            <linear_velocity_i_range>0 0</linear_velocity_i_range>
-            <!-- output -->
+        <plugin name='diff_drive' filename='libgazebo_ros_diff_drive.so'>
+            <!-- Wheel Information -->
+            <left_joint>left_wheel_joint</left_joint>
+            <right_joint>right_wheel_joint</right_joint>
+            <wheel_separation>0.35</wheel_separation>
+            <wheel_diameter>0.1</wheel_diameter>
+            <!-- Limits -->
+            <max_wheel_torque>200</max_wheel_torque>
+            <max_wheel_acceleration>10.0</max_wheel_acceleration>
+            <!-- Output -->
+            <odometry_frame>odom</odometry_frame>
+            <robot_base_frame>base_link</robot_base_frame>
             <publish_odom>true</publish_odom>
             <publish_odom_tf>true</publish_odom_tf>
             <publish_wheel_tf>true</publish_wheel_tf>
-            <publish_distance>true</publish_distance>
-            <odometry_frame>odom_demo</odometry_frame>
-            <robot_base_frame>chassis</robot_base_frame>
-            </plugin>
+        </plugin>
+    </gazebo>
 </robot>

File: description/robot_core.xacro (robot description, xacro)
@@ -21,39 +21,36 @@
         <parent link="base_link"/>
         <child link="chassis"/>
-        <origin xyz="-0.05 0 0"/>
+        <origin xyz="-0.1 0 0"/>
     </joint>
     <link name="chassis">
         <visual>
-            <origin xyz="0.105 0 0.0625" rpy="0 0 0"/>
+            <origin xyz="0.15 0 0.075" rpy="0 0 0"/>
             <geometry>
-                <box size="0.21 0.085 0.125"/>
+                <box size="0.3 0.3 0.15"/>
             </geometry>
             <material name="white"/>
         </visual>
         <collision>
-            <origin xyz="0.105 0 0.0625" rpy="0 0 0"/>
+            <origin xyz="0.15 0 0.075" rpy="0 0 0"/>
             <geometry>
-                <box size="0.21 0.085 0.125"/>
+                <box size="0.3 0.3 0.15"/>
             </geometry>
+            <material name="white"/>
         </collision>
-        <xacro:inertial_box mass="0.5" x="0.105" y="0" z="0.0625">
-            <origin xyz="0.105 0 0.0625" rpy="0 0 0"/>
-        </xacro:inertial_box>
     </link>
     <gazebo reference="chassis">
         <material>Gazebo/White</material>
     </gazebo>
-    <!-- WHEELS -->
-    <!-- REAR LEFT WHEEL -->
-    <joint name="rear_left_wheel_joint" type="continuous">
+    <!-- LEFT WHEEL -->
+    <joint name="left_wheel_joint" type="continuous">
         <parent link="base_link"/>
-        <child link="rear_left_wheel"/>
-        <origin xyz="0 0.0425 0" rpy="-${pi/2} 0 0"/>
+        <child link="left_wheel"/>
+        <origin xyz="0 0.175 0" rpy="-${pi/2} 0 0"/>
         <axis xyz="0 0 1"/>
     </joint>
-    <link name="rear_left_wheel">
+    <link name="left_wheel">
         <visual>
             <geometry>
-                <cylinder length="0.026" radius="0.03" />
+                <cylinder length="0.04" radius="0.05" />
             </geometry>
             <material name="blue"/>
@@ -61,25 +58,26 @@
         <collision>
             <geometry>
-                <cylinder length="0.026" radius="0.03" />
+                <cylinder length="0.04" radius="0.05" />
             </geometry>
+            <material name="blue"/>
         </collision>
-        <xacro:inertial_cylinder mass="0.1" radius="0.03" length="0.026">
-            <origin xyz="0 0 0" rpy="-${pi/2} 0 0"/>
+        <xacro:inertial_cylinder mass="0.1" radius="0.05" length="0.04">
+            <origin xyz="0 0 0" rpy="0 0 0"/>
         </xacro:inertial_cylinder>
     </link>
-    <gazebo reference="rear_left_wheel">
+    <gazebo reference="left_wheel">
         <material>Gazebo/Blue</material>
     </gazebo>
-    <!-- REAR RIGHT WHEEL -->
-    <joint name="rear_right_wheel_joint" type="continuous">
+    <!-- RIGHT WHEEL -->
+    <joint name="right_wheel_joint" type="continuous">
         <parent link="base_link"/>
-        <child link="rear_right_wheel"/>
-        <origin xyz="0 -0.0425 0" rpy="${pi/2} 0 0"/>
+        <child link="right_wheel"/>
+        <origin xyz="0 -0.175 0" rpy="${pi/2} 0 0"/>
         <axis xyz="0 0 -1"/>
     </joint>
-    <link name="rear_right_wheel">
+    <link name="right_wheel">
         <visual>
             <geometry>
-                <cylinder length="0.026" radius="0.03" />
+                <cylinder length="0.04" radius="0.05" />
             </geometry>
             <material name="blue"/>
@@ -87,65 +85,42 @@
         <collision>
             <geometry>
-                <cylinder length="0.026" radius="0.03" />
+                <cylinder length="0.04" radius="0.05" />
             </geometry>
+            <material name="blue"/>
         </collision>
-        <xacro:inertial_cylinder mass="0.1" radius="0.03" length="0.026">
-            <origin xyz="0 0 0" rpy="-${pi/2} 0 0"/>
+        <xacro:inertial_cylinder mass="0.1" radius="0.05" length="0.04">
+            <origin xyz="0 0 0" rpy="0 0 0"/>
         </xacro:inertial_cylinder>
     </link>
-    <gazebo reference="rear_right_wheel">
+    <gazebo reference="right_wheel">
         <material>Gazebo/Blue</material>
     </gazebo>
-    <!-- FRONT LEFT WHEEL -->
-    <joint name="front_left_wheel_joint" type="continuous">
-        <parent link="base_link"/>
-        <child link="front_left_wheel"/>
-        <origin xyz="0.1 0.0425 0" rpy="-${pi/2} 0 0"/>
-        <axis xyz="0 0 1"/>
+    <!-- CASTER WHEEL -->
+    <joint name="caster_wheel_joint" type="fixed">
+        <parent link="chassis"/>
+        <child link="caster_wheel"/>
+        <origin xyz="0.24 0 0" rpy="0 0 0"/>
     </joint>
-    <link name="front_left_wheel">
+    <link name="caster_wheel">
         <visual>
             <geometry>
-                <cylinder length="0.026" radius="0.03" />
+                <sphere radius="0.05" />
             </geometry>
-            <material name="orange"/>
+            <material name="black"/>
         </visual>
         <collision>
             <geometry>
-                <cylinder length="0.026" radius="0.03" />
+                <sphere radius="0.05" />
             </geometry>
+            <material name="black"/>
         </collision>
-        <xacro:inertial_cylinder mass="0.1" radius="0.03" length="0.026">
-            <origin xyz="0 0 0" rpy="-${pi/2} 0 0"/>
-        </xacro:inertial_cylinder>
+        <xacro:inertial_sphere mass="0.1" radius="0.05">
+            <origin xyz="0 0 0" rpy="0 0 0"/>
+        </xacro:inertial_sphere>
     </link>
-    <gazebo reference="front_left_wheel">
-        <material>Gazebo/Orange</material>
-    </gazebo>
-    <!-- FRONT RIGHT WHEEL -->
-    <joint name="front_right_wheel_joint" type="continuous">
-        <parent link="base_link"/>
-        <child link="front_right_wheel"/>
-        <origin xyz="0.1 -0.0425 0" rpy="${pi/2} 0 0"/>
-        <axis xyz="0 0 -1"/>
-    </joint>
-    <link name="front_right_wheel">
-        <visual>
-            <geometry>
-                <cylinder length="0.026" radius="0.03" />
-            </geometry>
-            <material name="orange"/>
-        </visual>
-        <collision>
-            <geometry>
-                <cylinder length="0.026" radius="0.03" />
-            </geometry>
-        </collision>
-        <xacro:inertial_cylinder mass="0.1" radius="0.03" length="0.026">
-            <origin xyz="0 0 0" rpy="-${pi/2} 0 0"/>
-        </xacro:inertial_cylinder>
-    </link>
-    <gazebo reference="front_right_wheel">
-        <material>Gazebo/Orange</material>
+    <gazebo reference="caster_wheel">
+        <material>Gazebo/Black</material>
+        <mu1 value="0.001"/>
+        <mu2 value="0.001"/>
     </gazebo>
 </robot>
