Commit message: URDF files updated

File: description/robot_core.xacro (robot description, xacro)
@@ -41,4 +41,7 @@
         </xacro:inertial_box>
     </link>
+    <gazebo reference="chassis">
+        <material>Gazebo/White</material>
+    </gazebo>
     <!-- WHEELS -->
     <!-- REAR LEFT WHEEL -->
@@ -65,4 +68,7 @@
         </xacro:inertial_cylinder>
     </link>
+    <gazebo reference="rear_left_wheel">
+        <material>Gazebo/Blue</material>
+    </gazebo>
     <!-- REAR RIGHT WHEEL -->
     <joint name="rear_right_wheel_joint" type="continuous">
@@ -88,12 +94,15 @@
         </xacro:inertial_cylinder>
     </link>
+    <gazebo reference="rear_right_wheel">
+        <material>Gazebo/Blue</material>
+    </gazebo>
     <!-- FRONT LEFT WHEEL -->
-    <joint name="front__left_wheel_joint" type="continuous">
+    <joint name="front_left_wheel_joint" type="continuous">
         <parent link="base_link"/>
-        <child link="front__left_wheel"/>
+        <child link="front_left_wheel"/>
         <origin xyz="0.1 0.0425 0" rpy="-${pi/2} 0 0"/>
         <axis xyz="0 0 1"/>
     </joint>
-    <link name="front__left_wheel">
+    <link name="front_left_wheel">
         <visual>
             <geometry>
@@ -111,12 +120,15 @@
         </xacro:inertial_cylinder>
     </link>
+    <gazebo reference="front_left_wheel">
+        <material>Gazebo/Orange</material>
+    </gazebo>
     <!-- FRONT RIGHT WHEEL -->
-    <joint name="front__right_wheel_joint" type="continuous">
+    <joint name="front_right_wheel_joint" type="continuous">
         <parent link="base_link"/>
-        <child link="front__right_wheel"/>
+        <child link="front_right_wheel"/>
         <origin xyz="0.1 -0.0425 0" rpy="${pi/2} 0 0"/>
         <axis xyz="0 0 -1"/>
     </joint>
-    <link name="front__right_wheel">
+    <link name="front_right_wheel">
         <visual>
             <geometry>
@@ -134,3 +146,6 @@
         </xacro:inertial_cylinder>
     </link>
+    <gazebo reference="front_right_wheel">
+        <material>Gazebo/Orange</material>
+    </gazebo>
 </robot>

Commit message: lidar.xacro added

File: description/robot_core.xacro (robot description, xacro)
@@ -13,4 +13,7 @@
     <material name="black">
         <color rgba="0 0 0 1"/>
+    </material>
+    <material name="red">
+        <color rgba="1 0 0 1"/>
     </material>
     <!-- BASE LINK -->
@@ -121,6 +124,6 @@
     <gazebo reference="caster_wheel">
         <material>Gazebo/Black</material>
-        <mu1 value="0.001"/>
-        <mu2 value="0.001"/>
+        <mu1 value="0.01"/>
+        <mu2 value="0.01"/>
     </gazebo>
 </robot>
